Commit message: target done

File: cartographer_ros/cartographer_ros/urdf/backpack_2d.urdf (robot description, URDF)
Before this commit: robot cartographer_backpack_2d, 4 links, 3 joints
Links:
- removed link base_link
- removed link horizontal_laser_link
- removed link imu_link
- removed link vertical_laser_link
- added link target/base_link
- added link target/horizontal_laser_link; visual cylinder length=0.05 radius=0.03
- added link target/imu_link; visual box size=0.06 0.04 0.02
- added link target/vertical_laser_link; visual cylinder length=0.05 radius=0.03
Joints:
- removed joint horizontal_laser_link_joint
- removed joint imu_link_joint
- removed joint vertical_laser_link_joint
- added joint target/horizontal_laser_link_joint: type fixed, parent target/base_link, child target/horizontal_laser_link, origin xyz=0.1007 0 0.0558
- added joint target/imu_link_joint: type fixed, parent target/base_link, child target/imu_link, origin xyz=0 0 0
- added joint target/vertical_laser_link_joint: type fixed, parent target/base_link, child target/vertical_laser_link, origin xyz=0.1007 0 0.1814 rpy=0 -1.570796 3.141593
